Commit message: Add lidar simulation

File: rover_description/urdf/rover_a1.urdf.xacro (robot description, xacro)
@@ -2,6 +2,8 @@
 <robot name="rover_a1" xmlns:xacro="http://wiki.ros.org/xacro">
   <xacro:arg name="use_sim" default="false" />
-  <xacro:arg name="imu_xyz" default="0.052 0.073 -0.006" />
+  <xacro:arg name="imu_xyz" default="0.0 0.0 0.0" />
   <xacro:arg name="imu_rpy" default="0.0 0.0 -1.57" />
+  <xacro:arg name="lidar_xyz" default="0.0 0.0 0.0" />
+  <xacro:arg name="lidar_rpy" default="0.0 0.0 -1.57" />
   <xacro:arg name="wheel_config_file" default="$(find rover_description)/config/wheel_01.yaml" />
   <xacro:arg name="controller_config_file" default="$(find rover_controller)/config/wheel_01_controller.yaml" />
@@ -12,4 +14,6 @@
     imu_xyz="$(arg imu_xyz)"
     imu_rpy="$(arg imu_rpy)"
+    lidar_xyz="$(arg lidar_xyz)"
+    lidar_rpy="$(arg lidar_rpy)"
     wheel_config_file="$(arg wheel_config_file)"
     controller_config_file="$(arg controller_config_file)"

File: rover_description/urdf/rover_a1/base.urdf.xacro (robot description, xacro)
@@ -5,5 +5,7 @@
     params="wheel_radius
             imu_xyz
-            imu_rpy">
+            imu_rpy
+            lidar_xyz
+            lidar_rpy">
     <link name="base_link" />
     <joint name="base_to_body_joint" type="fixed">
@@ -31,4 +33,10 @@
     </joint>
     <link name="imu_link" />
+    <joint name="body_to_lidar_joint" type="fixed">
+      <origin xyz="${lidar_xyz}" rpy="${lidar_rpy}" />
+      <parent link="body_link" />
+      <child link="lidar_link" />
+    </joint>
+    <link name="lidar_link" />
     <joint name="body_to_footprint_joint" type="fixed">
       <origin xyz="0.0 0.0 -0.1359" rpy="0.0 0.0 0.0" />

File: rover_description/urdf/rover_a1/rover_a1_macro.urdf.xacro (robot description, xacro)
@@ -8,8 +8,12 @@
             imu_xyz:='0.0 0.0 0.0'
             imu_rpy:='0.0 0.0 0.0'
+            lidar_xyz:='0.0 0.0 0.0'
+            lidar_rpy:='0.0 0.0 0.0'
             namespace:=''">
     <xacro:if value="${use_sim}">
-      <xacro:property name="imu_xyz" value="0.052 0.073 -0.235" />
-      <xacro:property name="imu_rpy" value="0.0 0.0 -1.57" />
+      <xacro:property name="imu_xyz" value="0.0 0.0 0.0" />
+      <xacro:property name="imu_rpy" value="0.0 0.0 0.0" />
+      <xacro:property name="lidar_xyz" value="0.0 0.0 0.25" />
+      <xacro:property name="lidar_rpy" value="0.0 0.0 0.0" />
     </xacro:if>
     <xacro:property name="ns" value='${namespace + "/" if namespace else ""}' />
@@ -23,4 +27,6 @@
     <!-- IMU macros -->
     <xacro:include filename="$(find rover_description)/urdf/common/imu.urdf.xacro" ns="imu" />
+    <!-- Lidar macros -->
+    <xacro:include filename="$(find rover_description)/urdf/common/lidar.urdf.xacro" ns="lidar" />
     <!-- Gazebo system macros -->
     <xacro:include filename="$(find rover_description)/urdf/common/gazebo_system.urdf.xacro" ns="gazebo_system" />
@@ -29,5 +35,7 @@
       wheel_radius="${wheel_config['wheel_radius']}"
       imu_xyz="${imu_xyz}"
-      imu_rpy="${imu_rpy}" />
+      imu_rpy="${imu_rpy}"
+      lidar_xyz="${lidar_xyz}"
+      lidar_rpy="${lidar_rpy}" />
     <!-- Rover wheel -->
     <xacro:wheel.wheel
@@ -110,4 +118,6 @@
     <!-- Instantiate IMU -->
     <xacro:imu.imu use_sim="${use_sim}" reference_frame="imu_link" namespace="${namespace}" />
+    <!-- Instantiate LIDAR -->
+    <xacro:lidar.lidar use_sim="${use_sim}" reference_frame="lidar_link" namespace="${namespace}" />
     <xacro:if value="${use_sim}">
     <!-- Instantiate Gazebo System -->

Commit message: Set correct position of the IMU

File: rover_description/urdf/rover_a1.urdf.xacro (robot description, xacro)
@@ -3,7 +3,7 @@
   <xacro:arg name="use_sim" default="false" />
   <xacro:arg name="imu_xyz" default="0.0 0.0 0.0" />
-  <xacro:arg name="imu_rpy" default="0.0 0.0 -1.57" />
+  <xacro:arg name="imu_rpy" default="0.0 0.0 0.0" />
   <xacro:arg name="lidar_xyz" default="0.0 0.0 0.0" />
-  <xacro:arg name="lidar_rpy" default="0.0 0.0 -1.57" />
+  <xacro:arg name="lidar_rpy" default="0.0 0.0 0.0" />
   <xacro:arg name="wheel_config_file" default="$(find rover_description)/config/wheel_01.yaml" />
   <xacro:arg name="controller_config_file" default="$(find rover_controller)/config/wheel_01_controller.yaml" />

File: rover_description/urdf/rover_a1/rover_a1_macro.urdf.xacro (robot description, xacro)
@@ -12,7 +12,7 @@
             namespace:=''">
     <xacro:if value="${use_sim}">
-      <xacro:property name="imu_xyz" value="0.0 0.0 0.0" />
+      <xacro:property name="imu_xyz" value="0.26 0.0 0.18" />
       <xacro:property name="imu_rpy" value="0.0 0.0 0.0" />
-      <xacro:property name="lidar_xyz" value="0.0 0.0 0.25" />
+      <xacro:property name="lidar_xyz" value="0.0 0.0 0.0" />
       <xacro:property name="lidar_rpy" value="0.0 0.0 0.0" />
     </xacro:if>
