Commit message: Rework on rover_description

File: rover_description/urdf/rover_a1.urdf.xacro (robot description, xacro)
@@ -8,5 +8,6 @@
   <xacro:arg name="wheel_config_file" default="$(find rover_description)/config/wheel_01.yaml" />
   <xacro:arg name="battery_config_file" default="$(find rover_description)/config/battery.yaml" />
-  <xacro:arg name="controller_config_file" default="$(find rover_controller)/config/wheel_01_controller.yaml" />
+  <!-- Only used by the gz_ros2_control plugin (use_sim:=true); the caller must supply it. -->
+  <xacro:arg name="controller_config_file" default="" />
   <xacro:arg name="namespace" default="" />
   <xacro:include filename="$(find rover_description)/urdf/rover_a1/rover_a1_macro.urdf.xacro" ns="rover" />

File: rover_description/urdf/rover_a1/rover_a1_macro.urdf.xacro (robot description, xacro)
@@ -20,6 +20,6 @@
     <xacro:property name="ns" value='${namespace + "/" if namespace else ""}' />
     <xacro:property name="wheel_config" value="${xacro.load_yaml(wheel_config_file)}" />
-    <xacro:property name="wheelbase" value="0.2542" />
-    <xacro:property name="wheel_mount_point_y" value="0.31301" />
+    <xacro:property name="wheelbase" value="${wheel_config['wheelbase']}" />
+    <xacro:property name="wheel_mount_point_y" value="${wheel_config['wheel_separation'] / 2.0}" />
     <!-- Rover base macros -->
     <xacro:include filename="$(find rover_description)/urdf/rover_a1/base.urdf.xacro" ns="body" />
