Commit message: Integrate the RUTX11 GPS and EKF_USE_GPS localization mode
Add rover_gps: launches the nmea_navsat_driver socket driver for the NMEA
the RUTX11 forwards over UDP, reports GPS fix health on diagnostics, and
aligns the odom yaw to ENU from GNSS course to publish gps/heading_imu.

EKF_USE_GPS selects the localization: false keeps the wheels + IMU EKF;
true adds a global EKF (map -> odom) fusing odometry/gps from
navsat_transform. Wire rover_gps into rover_bringup, rover_metapackage
and the diagnostic aggregator, add gps_link to the URDF, and add a
script to configure the RUTX11 NMEA forwarding.

Co-Authored-By: Claude Opus 5 <noreply@anthropic.com>

File: rover_description/urdf/rover_a1.urdf.xacro (robot description, xacro)
@@ -6,4 +6,6 @@
   <xacro:arg name="lidar_xyz" default="0.0 0.0 0.0" />
   <xacro:arg name="lidar_rpy" default="0.0 0.0 0.0" />
+  <xacro:arg name="gps_xyz" default="0.0 0.0 0.0" />
+  <xacro:arg name="gps_rpy" default="0.0 0.0 0.0" />
   <xacro:arg name="wheel_config_file" default="$(find rover_description)/config/wheel_01.yaml" />
   <xacro:arg name="battery_config_file" default="$(find rover_description)/config/battery.yaml" />
@@ -18,4 +20,6 @@
     lidar_xyz="$(arg lidar_xyz)"
     lidar_rpy="$(arg lidar_rpy)"
+    gps_xyz="$(arg gps_xyz)"
+    gps_rpy="$(arg gps_rpy)"
     wheel_config_file="$(arg wheel_config_file)"
     battery_config_file="$(arg battery_config_file)"

File: rover_description/urdf/rover_a1/base.urdf.xacro (robot description, xacro)
@@ -8,5 +8,7 @@
             imu_rpy
             lidar_xyz
-            lidar_rpy">
+            lidar_rpy
+            gps_xyz
+            gps_rpy">
     <link name="base_link" />
     <joint name="base_to_body_joint" type="fixed">
@@ -40,4 +42,11 @@
     </joint>
     <link name="lidar_link" />
+    <!-- GNSS antenna of the RUTX11 (frame_id of gps/fix); navsat_transform uses this offset. -->
+    <joint name="body_to_gps_joint" type="fixed">
+      <origin xyz="${gps_xyz}" rpy="${gps_rpy}" />
+      <parent link="body_link" />
+      <child link="gps_link" />
+    </joint>
+    <link name="gps_link" />
     <!-- Ground projection of body_link: the wheel axis height minus the wheel radius. -->
     <joint name="body_to_footprint_joint" type="fixed">

File: rover_description/urdf/rover_a1/rover_a1_macro.urdf.xacro (robot description, xacro)
@@ -11,4 +11,6 @@
             lidar_xyz:='0.0 0.0 0.0'
             lidar_rpy:='0.0 0.0 0.0'
+            gps_xyz:='0.0 0.0 0.0'
+            gps_rpy:='0.0 0.0 0.0'
             namespace:=''">
     <xacro:if value="${use_sim}">
@@ -47,5 +49,7 @@
       imu_rpy="${imu_rpy}"
       lidar_xyz="${lidar_xyz}"
-      lidar_rpy="${lidar_rpy}" />
+      lidar_rpy="${lidar_rpy}"
+      gps_xyz="${gps_xyz}"
+      gps_rpy="${gps_rpy}" />
     <!-- Rover wheel -->
     <xacro:wheel.wheel

Commit message: rover_description: add camera_link for the RealSense D435i
Fixed joint from body_link, always present so the TF tree does not change when
the camera is toggled. The default pose (0.25 0 0.2, facing forward) is an
assumption until measured; override with ROVER_CAMERA_LOCALIZATION_* and
ROVER_CAMERA_ORIENTATION_*.

Co-Authored-By: Claude Sonnet 5.5 <noreply@anthropic.com>

File: rover_description/urdf/rover_a1.urdf.xacro (robot description, xacro)
@@ -8,4 +8,6 @@
   <xacro:arg name="gps_xyz" default="0.0 0.0 0.0" />
   <xacro:arg name="gps_rpy" default="0.0 0.0 0.0" />
+  <xacro:arg name="camera_xyz" default="0.25 0.0 0.2" />
+  <xacro:arg name="camera_rpy" default="0.0 0.0 0.0" />
   <xacro:arg name="wheel_config_file" default="$(find rover_description)/config/wheel_01.yaml" />
   <xacro:arg name="battery_config_file" default="$(find rover_description)/config/battery.yaml" />
@@ -22,4 +24,6 @@
     gps_xyz="$(arg gps_xyz)"
     gps_rpy="$(arg gps_rpy)"
+    camera_xyz="$(arg camera_xyz)"
+    camera_rpy="$(arg camera_rpy)"
     wheel_config_file="$(arg wheel_config_file)"
     battery_config_file="$(arg battery_config_file)"

File: rover_description/urdf/rover_a1/base.urdf.xacro (robot description, xacro)
@@ -11,4 +11,6 @@
             gps_xyz
             gps_rpy
+            camera_xyz:='0.25 0.0 0.2'
+            camera_rpy:='0.0 0.0 0.0'
             use_sim:=false">
     <!-- REP-105 root: ground projection of base_link. The odometry filters publish
@@ -83,4 +85,14 @@
     </joint>
     <link name="gps_link" />
+    <!-- RealSense D435i. camera_link is the driver's TF root (REP-103, x forward): the realsense
+         node publishes camera_link -> optical frames itself. Mount pose is an ASSUMPTION until
+         measured on the rover; override with ROVER_CAMERA_LOCALIZATION_* / ROVER_CAMERA_ORIENTATION_*.
+         The frame always exists so the TF tree does not change when ROVER_USE_CAMERA toggles. -->
+    <joint name="body_to_camera_joint" type="fixed">
+      <origin xyz="${camera_xyz}" rpy="${camera_rpy}" />
+      <parent link="body_link" />
+      <child link="camera_link" />
+    </joint>
+    <link name="camera_link" />
   </xacro:macro>
 </robot>

File: rover_description/urdf/rover_a1/rover_a1_macro.urdf.xacro (robot description, xacro)
@@ -13,4 +13,6 @@
             gps_xyz:='0.0 0.0 0.0'
             gps_rpy:='0.0 0.0 0.0'
+            camera_xyz:='0.25 0.0 0.2'
+            camera_rpy:='0.0 0.0 0.0'
             namespace:=''">
     <xacro:if value="${use_sim}">
@@ -63,4 +65,6 @@
       gps_xyz="${gps_xyz}"
       gps_rpy="${gps_rpy}"
+      camera_xyz="${camera_xyz}"
+      camera_rpy="${camera_rpy}"
       use_sim="${use_sim}" />
     <!-- Rover wheel -->

Commit message: rover_description, rover_gazebo: opt-in Gazebo depth camera (ROVER_USE_CAMERA)
With use_sim and ROVER_USE_CAMERA=true the URDF gets a Gazebo depth camera on camera_link
standing in for the RealSense D435i (424x240, 87 deg, 15 Hz, 0.3-6 m), and gz_bridge maps its
cloud to <ns>/camera/depth/points, the topic rover_perception_bringup publishes on the rover.
That feeds the Nav 2 depth costmap source and rover_follow_me's fmoc in simulation.

The assumed real camera mount (0.25 0 0.2) is inside the body mesh, so with the Gazebo camera
and no ROVER_CAMERA_* mount set, camera_link moves just ahead of the front face (0.43 0 0.32).
Without the camera, the URDF (sim and real) is unchanged.

Co-Authored-By: Claude Opus 5.5 <noreply@anthropic.com>

File: rover_description/urdf/rover_a1.urdf.xacro (robot description, xacro)
@@ -10,4 +10,6 @@
   <xacro:arg name="camera_xyz" default="0.25 0.0 0.2" />
   <xacro:arg name="camera_rpy" default="0.0 0.0 0.0" />
+  <!-- With use_sim: a Gazebo depth camera on camera_link (ROVER_USE_CAMERA, see rover_load_urdf). -->
+  <xacro:arg name="use_camera" default="false" />
   <xacro:arg name="wheel_config_file" default="$(find rover_description)/config/wheel_01.yaml" />
   <xacro:arg name="battery_config_file" default="$(find rover_description)/config/battery.yaml" />
@@ -26,4 +28,5 @@
     camera_xyz="$(arg camera_xyz)"
     camera_rpy="$(arg camera_rpy)"
+    use_camera="$(arg use_camera)"
     wheel_config_file="$(arg wheel_config_file)"
     battery_config_file="$(arg battery_config_file)"

File: rover_description/urdf/rover_a1/rover_a1_macro.urdf.xacro (robot description, xacro)
@@ -15,4 +15,5 @@
             camera_xyz:='0.25 0.0 0.2'
             camera_rpy:='0.0 0.0 0.0'
+            use_camera:=false
             namespace:=''">
     <xacro:if value="${use_sim}">
@@ -28,4 +29,12 @@
       <xacro:if value="${[float(v) for v in str(lidar_xyz).split()] == [0.0, 0.0, 0.0]}">
         <xacro:property name="lidar_xyz" value="0.0 0.0 0.68" />
+      </xacro:if>
+      <!-- Likewise the Gazebo camera (use_camera only, so other simulations keep camera_link
+           where it was): the assumed real mount (0.25 0 0.2, rover_load_urdf) is inside the body
+           mesh (x up to 0.413, top z = 0.30), where it would see only the body. Keep a
+           ROVER_CAMERA_* mount when one is set, else put it just ahead of the front face, above
+           the body top. -->
+      <xacro:if value="${use_camera and [float(v) for v in str(camera_xyz).split()] == [0.25, 0.0, 0.2]}">
+        <xacro:property name="camera_xyz" value="0.43 0.0 0.32" />
       </xacro:if>
     </xacro:if>
@@ -53,4 +62,6 @@
     <!-- GPS macros -->
     <xacro:include filename="$(find rover_description)/urdf/common/gps.urdf.xacro" ns="gps" />
+    <!-- Depth camera macros -->
+    <xacro:include filename="$(find rover_description)/urdf/common/depth_camera.urdf.xacro" ns="depth_camera" />
     <!-- Gazebo system macros -->
     <xacro:include filename="$(find rover_description)/urdf/common/gazebo_system.urdf.xacro" ns="gazebo_system" />
@@ -292,4 +303,7 @@
     <!-- Instantiate GPS -->
     <xacro:gps.gps use_sim="${use_sim}" reference_frame="gps_link" namespace="${namespace}" />
+    <!-- Instantiate the depth camera (Gazebo only, and only with ROVER_USE_CAMERA) -->
+    <xacro:depth_camera.depth_camera
+      use_sim="${use_sim and use_camera}" reference_frame="camera_link" namespace="${namespace}" />
     <xacro:if value="${use_sim}">
       <!-- Instantiate Battery -->
