Commit message: Fix wheel base. Xacro test

File: rover_description/urdf/common/wheel.urdf.xacro (robot description, xacro)
@@ -1,37 +1,32 @@
 <?xml version="1.0" encoding="utf-8"?>
 <robot xmlns:xacro="http://wiki.ros.org/xacro">
-  <xacro:macro name="wheel" params="config prefix mount_point_x mount_point_y">
+  <!-- REP-103 frame: +x forward, +y left, +z up.
+       fl = (+x,+y)  fr = (+x,-y)  rl = (-x,+y)  rr = (-x,-y)
+       All four wheels spin about +y, so a positive joint velocity drives forward. -->
+  <xacro:macro name="wheel" params="config prefix mount_point_x mount_point_y mount_point_z">
     <xacro:if value="${prefix == 'fl'}">
       <xacro:property name="x" value="${mount_point_x}" />
       <xacro:property name="y" value="${mount_point_y}" />
-      <xacro:property name="mount_point_offset" value="${config['mount_point_offset']}" />
       <xacro:property name="inertia_y_offset" value="${config['inertia_y_offset']}" />
-      <xacro:property name="fdir" value="1 -1 0" />
     </xacro:if>
     <xacro:if value="${prefix == 'fr'}">
       <xacro:property name="x" value="${mount_point_x}" />
       <xacro:property name="y" value="-${mount_point_y}" />
-      <xacro:property name="mount_point_offset" value="-${config['mount_point_offset']}" />
       <xacro:property name="inertia_y_offset" value="${-config['inertia_y_offset']}" />
-      <xacro:property name="fdir" value="1 1 0" />
     </xacro:if>
     <xacro:if value="${prefix == 'rl'}">
       <xacro:property name="x" value="-${mount_point_x}" />
       <xacro:property name="y" value="${mount_point_y}" />
-      <xacro:property name="mount_point_offset" value="${config['mount_point_offset']}" />
       <xacro:property name="inertia_y_offset" value="${config['inertia_y_offset']}" />
-      <xacro:property name="fdir" value="1 1 0" />
     </xacro:if>
     <xacro:if value="${prefix == 'rr'}">
       <xacro:property name="x" value="-${mount_point_x}" />
       <xacro:property name="y" value="-${mount_point_y}" />
-      <xacro:property name="mount_point_offset" value="-${config['mount_point_offset']}" />
       <xacro:property name="inertia_y_offset" value="${-config['inertia_y_offset']}" />
-      <xacro:property name="fdir" value="1 -1 0" />
     </xacro:if>
     <joint name="body_to_${prefix}_wheel_base_joint" type="fixed">
       <parent link="body_link" />
       <child link="${prefix}_wheel_base_link" />
-      <origin xyz="${x} ${y} 0.033" rpy="0.0 0.0 0.0" />
+      <origin xyz="${x} ${y} ${mount_point_z}" rpy="0.0 0.0 0.0" />
     </joint>
     <link name="${prefix}_wheel_base_link" />

File: rover_description/urdf/rover_a1/base.urdf.xacro (robot description, xacro)
@@ -4,4 +4,5 @@
     name="body"
     params="wheel_radius
+            wheel_mount_point_z
             imu_xyz
             imu_rpy
@@ -39,6 +40,7 @@
     </joint>
     <link name="lidar_link" />
+    <!-- Ground projection of body_link: the wheel axis height minus the wheel radius. -->
     <joint name="body_to_footprint_joint" type="fixed">
-      <origin xyz="0.0 0.0 -0.1359" rpy="0.0 0.0 0.0" />
+      <origin xyz="0.0 0.0 ${wheel_mount_point_z - wheel_radius}" rpy="0.0 0.0 0.0" />
       <parent link="body_link" />
       <child link="base_footprint" />

File: rover_description/urdf/rover_a1/rover_a1_macro.urdf.xacro (robot description, xacro)
@@ -20,6 +20,10 @@
     <xacro:property name="ns" value='${namespace + "/" if namespace else ""}' />
     <xacro:property name="wheel_config" value="${xacro.load_yaml(wheel_config_file)}" />
-    <xacro:property name="wheelbase" value="${wheel_config['wheelbase']}" />
+    <!-- wheelbase and wheel_separation are full centre-to-centre distances, so each
+         mount point sits at half of them (REP-103: +x forward, +y left, +z up). -->
+    <xacro:property name="wheel_mount_point_x" value="${wheel_config['wheelbase'] / 2.0}" />
     <xacro:property name="wheel_mount_point_y" value="${wheel_config['wheel_separation'] / 2.0}" />
+    <!-- Height of the wheel axis above body_link; also fixes the ground plane. -->
+    <xacro:property name="wheel_mount_point_z" value="0.033" />
     <!-- Rover base macros -->
     <xacro:include filename="$(find rover_description)/urdf/rover_a1/base.urdf.xacro" ns="body" />
@@ -39,4 +43,5 @@
     <xacro:body.body
       wheel_radius="${wheel_config['wheel_radius']}"
+      wheel_mount_point_z="${wheel_mount_point_z}"
       imu_xyz="${imu_xyz}"
       imu_rpy="${imu_rpy}"
@@ -46,24 +51,28 @@
     <xacro:wheel.wheel
       config="${wheel_config}"
-      mount_point_x="${wheelbase}"
+      mount_point_x="${wheel_mount_point_x}"
       mount_point_y="${wheel_mount_point_y}"
+      mount_point_z="${wheel_mount_point_z}"
       prefix="fl" />
     <!-- Rover wheel -->
     <xacro:wheel.wheel
       config="${wheel_config}"
-      mount_point_x="${wheelbase}"
+      mount_point_x="${wheel_mount_point_x}"
       mount_point_y="${wheel_mount_point_y}"
+      mount_point_z="${wheel_mount_point_z}"
       prefix="fr" />
     <!-- Rover wheel -->
     <xacro:wheel.wheel
       config="${wheel_config}"
-      mount_point_x="${wheelbase}"
+      mount_point_x="${wheel_mount_point_x}"
       mount_point_y="${wheel_mount_point_y}"
+      mount_point_z="${wheel_mount_point_z}"
       prefix="rl" />
     <!-- Rover wheel -->
     <xacro:wheel.wheel
       config="${wheel_config}"
-      mount_point_x="${wheelbase}"
+      mount_point_x="${wheel_mount_point_x}"
       mount_point_y="${wheel_mount_point_y}"
+      mount_point_z="${wheel_mount_point_z}"
       prefix="rr" />
     <!-- ROS2 Controller -->
