Commit message: Fix Foxglove not rendering the robot meshes
foxglove_bridge serves package:// assets only if the URI matches
asset_uri_allowlist. The upstream default spells the extensions
lowercase and is compiled with a case-sensitive std::regex, so every
mesh in the URDF was refused: they all ended in uppercase .STL. Neither
body_link nor the wheels have a primitive-shape visual to fall back on,
so the 3D panel had nothing to draw and showed only the TF frames.

Rename the five meshes to lowercase .stl and update the two references.
Also override asset_uri_allowlist so an uppercase extension is accepted
regardless. std::regex uses the ECMAScript grammar, which rejects the
inline (?i) flag, so the pattern spells each letter as a two-case
character class instead.

Note this only fixes asset fetching. As with RViz in 19a2453, the
Foxglove 3D panel also needs its URDF layer pointed at
/<namespace>/robot_description with a matching frame prefix, which
lives in the layout rather than in this repo.

Co-Authored-By: Claude Opus 5 <noreply@anthropic.com>

File: rover_description/urdf/common/wheel.urdf.xacro (robot description, xacro)
@@ -43,5 +43,5 @@
         <origin xyz="0.0 0.0 0.0" rpy="0.0 0.0 0.0" />
         <geometry>
-          <mesh filename="package://${config['mesh_package']}/${config['folder_path']}/${prefix}_wheel.STL" />
+          <mesh filename="package://${config['mesh_package']}/${config['folder_path']}/${prefix}_wheel.stl" />
         </geometry>
         <material name="">

File: rover_description/urdf/rover_a1/base.urdf.xacro (robot description, xacro)
@@ -20,5 +20,5 @@
       <visual>
         <geometry>
-          <mesh filename="package://rover_description/meshes/rover_a1/base.STL" />
+          <mesh filename="package://rover_description/meshes/rover_a1/base.stl" />
         </geometry>
       </visual>

Commit message: Align rover_description with the SolidWorks export (ROVER_1000_WATT_VARIANT)
Update the xacro model from solidworks_exported/ROVER_1000_WATT_VARIANT.SLDASM:
- Meshes: body from the export's base_link.STL, decimated 4x (31 MB -> 7.8 MB,
  bounding box kept within 0.03 mm); wheel meshes replaced, now centred on the tyre.
- Body inertial from the export CSV (35.65 kg, new CoM and tensor); wheels
  5.0741 kg with CAD inertia and a 2.4 mm inboard CoM. Total mass 43.45 -> 55.94 kg.
- Wheel axis height above body_link 0.029 -> 0.037363.
- Add tyre_radius (CAD 0.1699) to wheel_01.yaml for the wheel collision cylinder and
  the base_footprint height, so the tyres touch the ground plane. wheel_radius stays
  0.1651 as the rolling radius the real odometry is tuned on.
- Sim: two collision boxes for the new body (main body + front arch); default sim
  lidar raised 0.45 -> 0.68 so the -15 deg ring clears the arch (0.62 hit it in
  Gazebo); drive controller wheel_radius 0.1699 so sim wheel odometry matches the
  rigid CAD tyre (steady-state odom vs ground truth within 0.03 %).
- test_wheel_geometry checks the CAD axis height and tyre_radius use.

Co-Authored-By: Claude Opus 5.5 <noreply@anthropic.com>

File: rover_description/urdf/common/wheel.urdf.xacro (robot description, xacro)
@@ -53,5 +53,5 @@
         <origin xyz="0.0 0.0 0.0" rpy="-${pi/2} 0.0 0.0" />
         <geometry>
-          <cylinder radius="${config['wheel_radius']}" length="${config['wheel_width']}" />
+          <cylinder radius="${config['tyre_radius']}" length="${config['wheel_width']}" />
         </geometry>
       </collision>

File: rover_description/urdf/rover_a1/base.urdf.xacro (robot description, xacro)
@@ -28,25 +28,38 @@
     </joint>
     <link name="body_link">
+      <!-- base.stl is the SolidWorks base_link.STL (solidworks_exported/
+           ROVER_1000_WATT_VARIANT.SLDASM) decimated 4x; body_link is its CAD frame. -->
       <visual>
         <geometry>
           <mesh filename="package://rover_description/meshes/rover_a1/base.stl" />
         </geometry>
+        <material name="">
+          <color rgba="0.792156862745098 0.819607843137255 0.933333333333333 1" />
+        </material>
       </visual>
-      <!-- Simulation only: a box over the base.stl bounds (x +/-0.351, y +/-0.313,
-           z -0.015..0.241) so the body hits obstacles in Gazebo. Gazebo does not
-           self-collide a model's links, so it cannot fight the wheels. -->
+      <!-- Simulation only: boxes over the base.stl bounds so the body hits obstacles in
+           Gazebo - the main body (x -0.410..0.413, y +/-0.27, z -0.02..0.30) and the front
+           arch (x 0.161..0.251, y +/-0.253, z 0.30..0.555). Gazebo does not self-collide a
+           model's links, so they cannot fight the wheels. -->
       <xacro:if value="${use_sim}">
         <collision>
-          <origin xyz="0.0 0.0 0.113" rpy="0.0 0.0 0.0" />
+          <origin xyz="0.0015 0.0 0.14" rpy="0.0 0.0 0.0" />
           <geometry>
-            <box size="0.702 0.626 0.256" />
+            <box size="0.823 0.54 0.32" />
+          </geometry>
+        </collision>
+        <collision>
+          <origin xyz="0.206 0.0 0.4275" rpy="0.0 0.0 0.0" />
+          <geometry>
+            <box size="0.09 0.506 0.255" />
           </geometry>
         </collision>
       </xacro:if>
+      <!-- From the SolidWorks export (base_link row of solidworks_exported/.../urdf/*.csv). -->
       <inertial>
-        <origin xyz="-0.0352516654672473 0.000230769565957786 0.0766816513547671" rpy="0 0 0" />
-        <mass value="33.445952" />
-        <inertia ixx="0.233794970398492" ixy="-0.000820762950210979" ixz="1.94037912313266E-05"
-                 iyy="0.228604041647293" iyz="3.84951327810773E-08" izz="0.363260170153768" />
+        <origin xyz="0.0246948542048735 0.00173673823842259 0.103380099372497" rpy="0 0 0" />
+        <mass value="35.6474447622668" />
+        <inertia ixx="0.319501966637767" ixy="-0.000816646517455797" ixz="4.83728654778507E-06"
+                 iyy="0.310232207152549" iyz="-5.04256505510483E-05" izz="0.559515096198424" />
       </inertial>
     </link>

File: rover_description/urdf/rover_a1/rover_a1_macro.urdf.xacro (robot description, xacro)
@@ -18,10 +18,12 @@
       <xacro:property name="imu_rpy" value="0.0 0.0 0.0" />
       <!-- Keep the ROVER_LIDAR_* mount when one is set; with the all-zero default the
-           gpu_lidar would sit inside the body mesh (top at z = 0.241), so lift it above.
-           Its lowest ring (-15 deg) must clear the body's far corner (0.47 m out), which
-           needs >= 0.126 m above the top; 0.45 gives 0.21 m. Lower, the rover sees itself
-           and the costmaps mark obstacles inside the footprint. -->
+           gpu_lidar would sit inside the body mesh, so lift it above. Its lowest ring
+           (-15 deg) must clear the far corner of the front arch's top (z = 0.555 at
+           x 0.251, y +/-0.253, 0.356 m out), which needs >= 0.555 + 0.356 * tan(15 deg)
+           = 0.650, and the body's far corner (top z = 0.30, 0.52 m out), which needs
+           >= 0.44; 0.68 clears both (0.62 was verified to hit the arch in Gazebo). Lower,
+           the rover sees itself and the costmaps mark obstacles inside the footprint. -->
       <xacro:if value="${[float(v) for v in str(lidar_xyz).split()] == [0.0, 0.0, 0.0]}">
-        <xacro:property name="lidar_xyz" value="0.0 0.0 0.45" />
+        <xacro:property name="lidar_xyz" value="0.0 0.0 0.68" />
       </xacro:if>
     </xacro:if>
@@ -32,6 +34,7 @@
     <xacro:property name="wheel_mount_point_x" value="${wheel_config['wheelbase'] / 2.0}" />
     <xacro:property name="wheel_mount_point_y" value="${wheel_config['wheel_separation'] / 2.0}" />
-    <!-- Height of the wheel axis above body_link; also fixes the ground plane. -->
-    <xacro:property name="wheel_mount_point_z" value="0.029" />
+    <!-- Height of the wheel axis above body_link; also fixes the ground plane. From the
+         SolidWorks export (joint_*_* origin z in solidworks_exported/.../urdf/*.csv). -->
+    <xacro:property name="wheel_mount_point_z" value="0.037363" />
     <!-- Rover base macros -->
     <xacro:include filename="$(find rover_description)/urdf/rover_a1/base.urdf.xacro" ns="body" />
@@ -52,5 +55,5 @@
     <!-- Rover body -->
     <xacro:body.body
-      wheel_radius="${wheel_config['wheel_radius']}"
+      wheel_radius="${wheel_config['tyre_radius']}"
       wheel_mount_point_z="${wheel_mount_point_z}"
       imu_xyz="${imu_xyz}"

Commit message: rover_description, rover_platform_mbse, docs: follow the CAD wheel geometry and mass
rover_description:
- The tyre tread sits 1.71 mm inboard of each CAD wheel joint (tread band of
  the exported link_*.STL). New wheel_01.yaml tyre_y_offset offsets the wheel
  collision cylinder, so the contact patches are 0.6136 m apart instead of
  wheel_separation (0.617 m, the joint distance). test_wheel_geometry checks it.

rover_platform_mbse (rebuilt with build_all: 25 passed, 7 known deviations,
traceability 0 errors; SysML export validates):
- platform_parameters.json: wheel_separation 0.615 -> 0.617, wheel_mass
  2.5 -> 5.0741, new tyre_radius, tyre_y_offset, wheel_mount_point_z and
  body_mass; source lines re-read.
- SWR-CTL-005, SWR-DESC-003, -004, -012 updated to the CAD values (axis height
  0.037363 m, base height 0.132537 m, mounts at +/-0.3085 m, URDF mass
  57.2739 kg). SWR-CTL-005 records that the effective track is now
  0.617 x 1.659 = 1.0236 m against the 1.020 m calibration.
- sys_sr_compliance.json: SYS-SR-001 mass, SYS-SR-026 footprint
  (0.923 x 0.802 m), SYS-SR-028 tip-over (55 deg with the CAD CoM height
  0.215 m), and the SYS-SR-001 open question now asks to re-take the xlsx
  Mass Properties sheet.

docs: specification mass, CoM height, yaw inertia, tip-over angle and Nav 2
footprint from the 2026-10-07 CAD; open-items track width and MBSE rows.

The SYS-SR workbook (requirement-owner master) is unchanged.

Co-Authored-By: Claude Opus 5.5 <noreply@anthropic.com>

File: rover_description/urdf/common/wheel.urdf.xacro (robot description, xacro)
@@ -9,4 +9,5 @@
       <xacro:property name="y" value="${mount_point_y}" />
       <xacro:property name="inertia_y_offset" value="${config['inertia_y_offset']}" />
+      <xacro:property name="tyre_y_offset" value="${config['tyre_y_offset']}" />
     </xacro:if>
     <xacro:if value="${prefix == 'fr'}">
@@ -14,4 +15,5 @@
       <xacro:property name="y" value="-${mount_point_y}" />
       <xacro:property name="inertia_y_offset" value="${-config['inertia_y_offset']}" />
+      <xacro:property name="tyre_y_offset" value="${-config['tyre_y_offset']}" />
     </xacro:if>
     <xacro:if value="${prefix == 'rl'}">
@@ -19,4 +21,5 @@
       <xacro:property name="y" value="${mount_point_y}" />
       <xacro:property name="inertia_y_offset" value="${config['inertia_y_offset']}" />
+      <xacro:property name="tyre_y_offset" value="${config['tyre_y_offset']}" />
     </xacro:if>
     <xacro:if value="${prefix == 'rr'}">
@@ -24,4 +27,5 @@
       <xacro:property name="y" value="-${mount_point_y}" />
       <xacro:property name="inertia_y_offset" value="${-config['inertia_y_offset']}" />
+      <xacro:property name="tyre_y_offset" value="${-config['tyre_y_offset']}" />
     </xacro:if>
     <joint name="body_to_${prefix}_wheel_base_joint" type="fixed">
@@ -51,5 +55,5 @@
       </visual>
       <collision>
-        <origin xyz="0.0 0.0 0.0" rpy="-${pi/2} 0.0 0.0" />
+        <origin xyz="0.0 ${tyre_y_offset} 0.0" rpy="-${pi/2} 0.0 0.0" />
         <geometry>
           <cylinder radius="${config['tyre_radius']}" length="${config['wheel_width']}" />
