Commit message: rover_gazebo: simulated RS16 lidar + GNSS, orchestrator-aligned command path
Bring the Gazebo simulation in line with the rover and the orchestrator so
rover_navigation / rover_mission_manager run against it unchanged (apart from
use_sim_time).

- Lidar: RS16-like gpu_lidar (16 rings +/-15 deg, 360 deg at 0.5 deg,
  0.2-20 m, 10 Hz), bridged to <ns>/rslidar_points; <ns>/scan is sliced by
  pointcloud_to_laserscan with the real driver's +/-0.25 m band. Sim mount
  defaults to 0.30 m above body_link when ROVER_LIDAR_* is unset.
- GNSS: new sim-only navsat sensor on gps_link -> <ns>/gps/fix (NavSatFix);
  world gets the NavSat system. use_gps (ROVER_USE_GPS) now drives fuse_gps
  and publish_global_tf (ROVER_GPS_PUBLISH_MAP_TF) is passed through.
- Command path: run rover_twist_mux (mux + motion lock) as on the rover, with
  sim_gpio_state.py publishing an all-clear hardware_interface/gpio_state
  (e_stop parameter simulates a software E-Stop). GUI teleop now feeds the
  mux instead of cmd_vel. twist_mux is no longer a hardware-only dependency.
- Fixes: gz-sim plugin names in the world, namespaced IMU/lidar gz frame ids,
  no empty IMU <ros2_control> in sim, model name falls back to rover_a1,
  spawn pose args declared where used, drop unused build deps and the bogus
  env hook, headless flag accepts true/false.
- World: perimeter walls and obstacles for lidar, costmaps and SLAM.

Co-Authored-By: Claude Opus 5 (1M context) <noreply@anthropic.com>

File: rover_description/urdf/common/imu.urdf.xacro (robot description, xacro)
@@ -51,5 +51,5 @@
           <visualize>false</visualize>
           <enable_metrics>false</enable_metrics>
-          <gz_frame_id>imu_link</gz_frame_id>
+          <gz_frame_id>${ns}${reference_frame}</gz_frame_id>
           <imu>
             <orientation_reference_frame>
@@ -84,7 +84,8 @@
       </gazebo>
     </xacro:if>
-    <!-- ROS2 controller -->
+    <!-- ROS2 controller. Hardware only: in simulation the IMU interfaces live in the
+         GazeboSimSystem block, and an empty <ros2_control> would have no <hardware>. -->
+    <xacro:unless value="${use_sim}">
     <ros2_control name="${ns}rover_imu" type="sensor">
-      <xacro:unless value="${use_sim}">
         <hardware>
           <!-- Hardware IMU sensor interface  -->
@@ -111,6 +112,6 @@
         <!-- IMU interfaces -->
         <xacro:imu_interface use_sim="${use_sim}" namespace="${namespace}" />
-      </xacro:unless>
     </ros2_control>
+    </xacro:unless>
   </xacro:macro>
 </robot>

File: rover_description/urdf/common/lidar.urdf.xacro (robot description, xacro)
@@ -7,34 +7,43 @@
             namespace:=''">
     <xacro:property name="ns" value='${namespace + "/" if namespace else ""}' />
-    <!-- Gazebo LIDAR -->
+    <!-- Gazebo LIDAR: stands in for the RoboSense RS16 (rover_rs16_lidar in rover_sensors).
+         16 rings over +/-15 deg, 360 deg at 0.5 deg, 0.2-20 m, 10 Hz. Gazebo publishes the
+         cloud on <ns>lidar/points; the bridge maps it to <ns>rslidar_points and
+         pointcloud_to_laserscan slices <ns>scan out of it, as the real driver does. -->
     <xacro:if value="${use_sim}">
       <gazebo reference="${reference_frame}">
-        <sensor name='gpu_lidar' type='gpu_lidar'>"
-          <topic>lidar</topic>
+        <sensor name="${ns}lidar" type="gpu_lidar">
+          <topic>${ns}lidar</topic>
           <update_rate>10</update_rate>
-          <gz_frame_id>lidar_link</gz_frame_id>
-          <ray>
-              <scan>
-                  <horizontal>
-                      <samples>640</samples>
-                      <resolution>1</resolution>
-                      <min_angle>-1.396263</min_angle>
-                      <max_angle>1.396263</max_angle>
-                  </horizontal>
-                  <vertical>
-                      <samples>1</samples>
-                      <resolution>0.01</resolution>
-                      <min_angle>0</min_angle>
-                      <max_angle>0</max_angle>
-                  </vertical>
-              </scan>
-              <range>
-                  <min>0.08</min>
-                  <max>10.0</max>
-                  <resolution>0.01</resolution>
-              </range>
-          </ray>
+          <!-- Frames carry the namespace prefix (robot_state_publisher frame_prefix). -->
+          <gz_frame_id>${ns}${reference_frame}</gz_frame_id>
+          <lidar>
+            <scan>
+              <horizontal>
+                <samples>720</samples>
+                <resolution>1</resolution>
+                <min_angle>-3.141593</min_angle>
+                <max_angle>3.141593</max_angle>
+              </horizontal>
+              <vertical>
+                <samples>16</samples>
+                <resolution>1</resolution>
+                <min_angle>-0.261799</min_angle>
+                <max_angle>0.261799</max_angle>
+              </vertical>
+            </scan>
+            <range>
+              <min>0.2</min>
+              <max>20.0</max>
+              <resolution>0.01</resolution>
+            </range>
+            <noise>
+              <type>gaussian</type>
+              <mean>0.0</mean>
+              <stddev>0.01</stddev>
+            </noise>
+          </lidar>
           <always_on>1</always_on>
-          <visualize>true</visualize>
+          <visualize>false</visualize>
         </sensor>
       </gazebo>

File: rover_description/urdf/rover_a1/rover_a1_macro.urdf.xacro (robot description, xacro)
@@ -17,6 +17,9 @@
       <xacro:property name="imu_xyz" value="-0.09 0.0 0.2" />
       <xacro:property name="imu_rpy" value="0.0 0.0 0.0" />
-      <xacro:property name="lidar_xyz" value="0.0 0.0 0.0" />
-      <xacro:property name="lidar_rpy" value="0.0 0.0 0.0" />
+      <!-- Keep the ROVER_LIDAR_* mount when one is set; with the all-zero default the
+           gpu_lidar would sit inside the body mesh (top at z = 0.241), so lift it above. -->
+      <xacro:if value="${[float(v) for v in str(lidar_xyz).split()] == [0.0, 0.0, 0.0]}">
+        <xacro:property name="lidar_xyz" value="0.0 0.0 0.30" />
+      </xacro:if>
     </xacro:if>
     <xacro:property name="ns" value='${namespace + "/" if namespace else ""}' />
@@ -40,4 +43,6 @@
     <!-- Lidar macros -->
     <xacro:include filename="$(find rover_description)/urdf/common/lidar.urdf.xacro" ns="lidar" />
+    <!-- GPS macros -->
+    <xacro:include filename="$(find rover_description)/urdf/common/gps.urdf.xacro" ns="gps" />
     <!-- Gazebo system macros -->
     <xacro:include filename="$(find rover_description)/urdf/common/gazebo_system.urdf.xacro" ns="gazebo_system" />
@@ -189,4 +194,6 @@
     <!-- Instantiate LIDAR -->
     <xacro:lidar.lidar use_sim="${use_sim}" reference_frame="lidar_link" namespace="${namespace}" />
+    <!-- Instantiate GPS -->
+    <xacro:gps.gps use_sim="${use_sim}" reference_frame="gps_link" namespace="${namespace}" />
     <xacro:if value="${use_sim}">
       <!-- Instantiate Battery -->

Commit message: rover_description: drop the namespace prefix from the ros2_control component names
ros2_control names each hardware component's node after the component (with '/' replaced by
'_') and puts it in the controller manager's namespace. The "${ns}" prefix therefore doubled the
namespace: /rover/rover_rover_system_node and /rover/rover_rover_imu on the rover. They are now
/rover/rover_system_node and /rover/rover_imu, the names the docs already used. In simulation
gz_ros2_control creates the node at the root, so it is /rover_system_node there.

Nothing refers to the component names by their prefixed form. The generated URDF differs only in
the two names for every use_sim/namespace/use_camera combination.

SWR-DESC-006 and SWR-DESC-010 (SWRS_DESC.slreqx, the JSON seed and the SysML export) say the
names carry no namespace prefix. The xlsx exports are regenerated in the next commit.

Co-Authored-By: Claude Opus 5.5 <noreply@anthropic.com>

File: rover_description/urdf/common/imu.urdf.xacro (robot description, xacro)
@@ -85,7 +85,8 @@
     </xacro:if>
     <!-- ROS2 controller. Hardware only: in simulation the IMU interfaces live in the
-         GazeboSimSystem block, and an empty <ros2_control> would have no <hardware>. -->
+         GazeboSimSystem block, and an empty <ros2_control> would have no <hardware>.
+         Unprefixed name, like rover_system_node: the node is /<namespace>/rover_imu. -->
     <xacro:unless value="${use_sim}">
-    <ros2_control name="${ns}rover_imu" type="sensor">
+    <ros2_control name="rover_imu" type="sensor">
         <hardware>
           <!-- Hardware IMU sensor interface  -->

File: rover_description/urdf/rover_a1/rover_a1_macro.urdf.xacro (robot description, xacro)
@@ -39,5 +39,4 @@
       </xacro:if>
     </xacro:if>
-    <xacro:property name="ns" value='${namespace + "/" if namespace else ""}' />
     <xacro:property name="wheel_config" value="${xacro.load_yaml(wheel_config_file)}" />
     <!-- wheelbase and wheel_separation are full centre-to-centre distances, so each
@@ -107,6 +106,7 @@
       mount_point_z="${wheel_mount_point_z}"
       prefix="rr" />
-    <!-- ROS2 Controller -->
-    <ros2_control name="${ns}rover_system_node" type="system">
+    <!-- ROS2 Controller. No namespace prefix in the name: ros2_control names the component's
+         node after it, inside the controller manager's namespace (/rover/rover_system_node). -->
+    <ros2_control name="rover_system_node" type="system">
       <!-- Joints -->
       <joint name="fl_wheel_base_to_fl_wheel_joint">
