Commit message: rover_description: raise sim lidar default mount to 0.45 m
At 0.30 m above body_link the RS16 stand-in's -15 deg ring hit the body
top (573 of 709 scan hits within 0.41 m). The costmaps marked obstacles
inside the footprint and MPPI stopped short of goals ("Optimizer fail to
compute path"). 0.45 m clears the body's far corner; self-hits are now 0
and Nav2 reaches goals in odom, slam and gps modes.

Co-Authored-By: Claude Opus 5 (1M context) <noreply@anthropic.com>

File: rover_description/urdf/rover_a1/rover_a1_macro.urdf.xacro (robot description, xacro)
@@ -18,7 +18,10 @@
       <xacro:property name="imu_rpy" value="0.0 0.0 0.0" />
       <!-- Keep the ROVER_LIDAR_* mount when one is set; with the all-zero default the
-           gpu_lidar would sit inside the body mesh (top at z = 0.241), so lift it above. -->
+           gpu_lidar would sit inside the body mesh (top at z = 0.241), so lift it above.
+           Its lowest ring (-15 deg) must clear the body's far corner (0.47 m out), which
+           needs >= 0.126 m above the top; 0.45 gives 0.21 m. Lower, the rover sees itself
+           and the costmaps mark obstacles inside the footprint. -->
       <xacro:if value="${[float(v) for v in str(lidar_xyz).split()] == [0.0, 0.0, 0.0]}">
-        <xacro:property name="lidar_xyz" value="0.0 0.0 0.30" />
+        <xacro:property name="lidar_xyz" value="0.0 0.0 0.45" />
       </xacro:if>
     </xacro:if>
