Commit message: Update IMU pose

File: rover_description/urdf/rover_a1/rover_a1_macro.urdf.xacro (robot description, xacro)
@@ -13,5 +13,5 @@
             namespace:=''">
     <xacro:if value="${use_sim}">
-      <xacro:property name="imu_xyz" value="0.26 0.0 0.18" />
+      <xacro:property name="imu_xyz" value="-0.09 0.0 0.2" />
       <xacro:property name="imu_rpy" value="0.0 0.0 0.0" />
       <xacro:property name="lidar_xyz" value="0.0 0.0 0.0" />

Commit message: Updare mount pose and wheel separation dist

File: rover_description/urdf/rover_a1/rover_a1_macro.urdf.xacro (robot description, xacro)
@@ -33,5 +33,5 @@
     <xacro:property name="wheel_mount_point_y" value="${wheel_config['wheel_separation'] / 2.0}" />
     <!-- Height of the wheel axis above body_link; also fixes the ground plane. -->
-    <xacro:property name="wheel_mount_point_z" value="0.033" />
+    <xacro:property name="wheel_mount_point_z" value="0.029" />
     <!-- Rover base macros -->
     <xacro:include filename="$(find rover_description)/urdf/rover_a1/base.urdf.xacro" ns="body" />
