Commit message: rover_description: make base_footprint the TF root (REP-105)
base_footprint hung off body_link, giving odom -> base_link -> body_link
-> base_footprint. With two_d_mode the EKF pinned base_link to z=0, so
odom sat one wheel radius (0.132 m) above the ground.

- URDF: base_footprint is the root; footprint_to_base_joint lifts
  base_link by wheel_radius - wheel_mount_point_z.
- EKFs (local + global) and the drive controller use base_footprint as
  the robot frame, so odom -> base_footprint is published.
- Gazebo: world -> odom at z=0; the spawn z is only the drop height.

Co-Authored-By: Claude Opus 5 (1M context) <noreply@anthropic.com>

File: rover_description/urdf/rover_a1/base.urdf.xacro (robot description, xacro)
@@ -11,4 +11,13 @@
             gps_xyz
             gps_rpy">
+    <!-- REP-105 root: ground projection of base_link. The odometry filters publish
+         odom -> base_footprint, so in 2D mode odom stays on the ground plane. -->
+    <link name="base_footprint" />
+    <!-- base_link sits above the ground by the wheel radius minus the axis offset. -->
+    <joint name="footprint_to_base_joint" type="fixed">
+      <origin xyz="0.0 0.0 ${wheel_radius - wheel_mount_point_z}" rpy="0.0 0.0 0.0" />
+      <parent link="base_footprint" />
+      <child link="base_link" />
+    </joint>
     <link name="base_link" />
     <joint name="base_to_body_joint" type="fixed">
@@ -49,11 +58,4 @@
     </joint>
     <link name="gps_link" />
-    <!-- Ground projection of body_link: the wheel axis height minus the wheel radius. -->
-    <joint name="body_to_footprint_joint" type="fixed">
-      <origin xyz="0.0 0.0 ${wheel_mount_point_z - wheel_radius}" rpy="0.0 0.0 0.0" />
-      <parent link="body_link" />
-      <child link="base_footprint" />
-    </joint>
-    <link name="base_footprint" />
   </xacro:macro>
 </robot>

Commit message: rover_gazebo: add rover_sim.sh launcher, sim-only body collision
- scripts/rover_sim.sh runs the simulation from a fresh terminal regardless
  of ~/.bashrc: ROVER_ROS_BUILD_TYPE=simulation, drops ZENOH_CONFIG_OVERRIDE
  (never joins the rover's router), starts a zenoh router bound to
  127.0.0.1:7447 and stops it on exit, stops a stale ros2 daemon, checks the
  apt dependencies, optional --build. Sourced, it only prepares the shell for
  a second terminal (orchestrator, ros2 CLI). Installed with the package.
- rover_description: body_link gets a box collision over the base.stl bounds
  in simulation only, so the body hits obstacles in Gazebo. The hardware URDF
  is unchanged.

Co-Authored-By: Claude Opus 5 (1M context) <noreply@anthropic.com>

File: rover_description/urdf/rover_a1/base.urdf.xacro (robot description, xacro)
@@ -10,5 +10,6 @@
             lidar_rpy
             gps_xyz
-            gps_rpy">
+            gps_rpy
+            use_sim:=false">
     <!-- REP-105 root: ground projection of base_link. The odometry filters publish
          odom -> base_footprint, so in 2D mode odom stays on the ground plane. -->
@@ -32,4 +33,15 @@
         </geometry>
       </visual>
+      <!-- Simulation only: a box over the base.stl bounds (x +/-0.351, y +/-0.313,
+           z -0.015..0.241) so the body hits obstacles in Gazebo. Gazebo does not
+           self-collide a model's links, so it cannot fight the wheels. -->
+      <xacro:if value="${use_sim}">
+        <collision>
+          <origin xyz="0.0 0.0 0.113" rpy="0.0 0.0 0.0" />
+          <geometry>
+            <box size="0.702 0.626 0.256" />
+          </geometry>
+        </collision>
+      </xacro:if>
       <inertial>
         <origin xyz="-0.0352516654672473 0.000230769565957786 0.0766816513547671" rpy="0 0 0" />

File: rover_description/urdf/rover_a1/rover_a1_macro.urdf.xacro (robot description, xacro)
@@ -56,5 +56,6 @@
       lidar_rpy="${lidar_rpy}"
       gps_xyz="${gps_xyz}"
-      gps_rpy="${gps_rpy}" />
+      gps_rpy="${gps_rpy}"
+      use_sim="${use_sim}" />
     <!-- Rover wheel -->
     <xacro:wheel.wheel

Commit message: rover_description, rover_platform_mbse, docs: follow the corrected CAD masses
The SolidWorks audit found wrong materials and unsourced masses in the CAD. They are now fixed in
the CAD repo:
- LATERAL_4mm_AL x2 is aluminium (was an unresolved "Steel" weighed at 1000 kg/m3)
- the plexiglass battery box is acrylic
- the 8 mm flanges are 6061 aluminium (were alloy steel)
- RUTX11 is 456 g (distributor spec)
- the battery is 5 kg (owner value)
- the hidden Box in MOTOR_DRIVER is removed (not on the real rover)

CAD total: 58.72 kg (SYS-SR-001 limit 60 kg).

body_link and wheel inertials are now computed from the per-part SolidWorks mass properties, not
the sw2urdf export. The exporter ignores mass overrides, and its body inertia (izz 0.57 kg m^2)
cannot add up to the assembly's 6.19 kg m^2 yaw inertia. The computed values match the assembly
to 2e-6, so the -0.2522 kg hand correction is gone.
- body_link: 39.5373 kg, izz 3.034
- wheel: 4.79607 kg

URDF total 58.72158 kg.

Synced: specification (mass, CoM height 0.218 m, yaw inertia 6.19, wheel mass), index, open-items,
platform_parameters, sys_sr_compliance, and SWR-DESC-012. Regenerated with build_all: 25 passed,
7 known deviations, 0 unexpected. The SysML export validates OK.

Co-Authored-By: Claude Opus 5.5 <noreply@anthropic.com>

File: rover_description/urdf/rover_a1/base.urdf.xacro (robot description, xacro)
@@ -58,15 +58,17 @@
         </collision>
       </xacro:if>
-      <!-- From the SolidWorks export (base_link row of solidworks_exported/.../urdf/*.csv),
-           except the mass. The exporter ignores user-overridden part masses and weighs the 4
-           DCC1000 motor controllers at their 1060 Alloy material mass (141.9 g) instead of
-           the 78.8 g override (an ASSUMPTION in the CAD, not weighed). Mass = exported
-           37.2298 - 4 x 0.06306 = 36.9775 kg, matching the CAD assembly (57.274 kg total).
-           CoM and inertia are left as exported (error well below 1 %). -->
+      <!-- Computed from the SolidWorks part mass properties of ROVER_1000_WATT_VARIANT
+           (2026-10-08): every part except the 4 WHEEL_CHUNK sub-assemblies, combined about
+           their joint CoM. The result matches the assembly's own mass properties (58.722 kg
+           total, yaw inertia 6.19 kg·m²) to 2e-6. This honours the CAD mass overrides, which
+           the sw2urdf exporter ignores: DCC1000 78.8 g (ASSUMPTION), RUTX11 456 g (distributor
+           spec), LiFePO4 5 kg (owner value). The exporter's body inertia (izz 0.57) is
+           also too small to add up to the assembly's 6.19 kg·m² yaw inertia, so it is not
+           used. -->
       <inertial>
-        <origin xyz="0.0160214617664491 -0.000470435452859783 0.107817531003205" rpy="0 0 0" />
-        <mass value="36.9775262386666" />
-        <inertia ixx="0.327697897335902" ixy="-0.000815380156152649" ixz="3.69646892519238E-06"
-                 iyy="0.314462293606544" iyz="-5.45800544682604E-05" izz="0.57169437099185" />
+        <origin xyz="0.014282 0.000997148 0.108927" rpy="0 0 0" />
+        <mass value="39.5373" />
+        <inertia ixx="1.52291" ixy="0.00251836" ixz="-0.0356428"
+                 iyy="2.29298" iyz="0.000836665" izz="3.03359" />
       </inertial>
     </link>

Commit message: rover_description, rover_platform_mbse, docs: follow the CAD clash fixes
The CAD clash fixes changed the mass (CAD repo 032673d, 4f95bff):
- the battery model is 163.5 mm deep, to fit the plexiglass box
- a 60 x 60 switch opening in the rear panel
- a D36 notch in the two bottom-front 149 mm profiles
- a D22 x 3 recess in the 17 mm wheel flanges

CAD total is now 58.674 kg (-47 g), yaw inertia 6.18 kg m^2, CoM still 0.218 m above the ground.

Recomputed from the per-part SolidWorks mass properties, now configuration-aware for the Notched
profile. They match the assembly to 3e-6 kg, 5e-8 m and 2e-6 kg m^2.
- body_link: 39.5026 kg, CoM 0.0146114 0.000906667 0.108928, izz 3.02892
- wheel: 4.79294 kg, ixx/izz 0.036460, iyy 0.065711, y offset -0.0026831

URDF total 58.67436 kg.

Synced: specification, open-items, platform_parameters, sys_sr_compliance and SWR-DESC-012.
build_all: 25 passed, 7 known deviations, 0 unexpected. The SysML export validates OK.

Co-Authored-By: Claude Opus 5.5 <noreply@anthropic.com>

File: rover_description/urdf/rover_a1/base.urdf.xacro (robot description, xacro)
@@ -59,16 +59,16 @@
       </xacro:if>
       <!-- Computed from the SolidWorks part mass properties of ROVER_1000_WATT_VARIANT
-           (2026-10-08): every part except the 4 WHEEL_CHUNK sub-assemblies, combined about
-           their joint CoM. The result matches the assembly's own mass properties (58.722 kg
-           total, yaw inertia 6.19 kg·m²) to 2e-6. This honours the CAD mass overrides, which
+           (2026-10-08, after the clash fixes): every part except the 4 WHEEL_CHUNK sub-assemblies, combined about
+           their joint CoM. The result matches the assembly's own mass properties (58.674 kg
+           total, yaw inertia 6.18 kg·m²) to 2e-6. This honours the CAD mass overrides, which
            the sw2urdf exporter ignores: DCC1000 78.8 g (ASSUMPTION), RUTX11 456 g (distributor
            spec), LiFePO4 5 kg (owner value). The exporter's body inertia (izz 0.57) is
-           also too small to add up to the assembly's 6.19 kg·m² yaw inertia, so it is not
+           also too small to add up to the assembly's 6.18 kg·m² yaw inertia, so it is not
            used. -->
       <inertial>
-        <origin xyz="0.014282 0.000997148 0.108927" rpy="0 0 0" />
-        <mass value="39.5373" />
-        <inertia ixx="1.52291" ixy="0.00251836" ixz="-0.0356428"
-                 iyy="2.29298" iyz="0.000836665" izz="3.03359" />
+        <origin xyz="0.0146114 0.000906667 0.108928" rpy="0 0 0" />
+        <mass value="39.5026" />
+        <inertia ixx="1.52214" ixy="0.00121013" ixz="-0.0357691"
+                 iyy="2.28896" iyz="0.000896478" izz="3.02892" />
       </inertial>
     </link>
